File: Stepcraft2-model600/relays/CNC-relays/CNC-relays.kicad_pcb (KiCad board)
At the start: 2 copper layers, 94 x 87.6 mm, 100 parts, among them J1 PC-GK2.1, J10 Conn_01x03_Pin, J11 Conn_01x01, J12 Conn_01x10_Pin, J13 Conn_01x04, J14 Conn_01x08, J15 Conn_02x02_Odd_Even, J16 Conn_02x02_Odd_Even, J17 Conn_02x02_Odd_Even, J18 Conn_02x02_Odd_Even, J19 Conn_02x02_Odd_Even, J2 Conn_02x04_Odd_Even, J20 Conn_02x02_Odd_Even, J21 Conn_02x02_Odd_Even, J22 Conn_02x02_Odd_Even, J23 Conn_01x02_Pin, J24 Conn_01x10_Pin, J25 Conn_01x01, J3 Conn_02x04_Odd_Even, J4 Conn_01x01, J5 FTDI breakout, J6 Conn_01x03, J7 Conn_01x03, J8 Conn_01x03, J9 Conn_01x03, U1 WT32-ETH01, U2 N7803-1PH, U3 THVD1400DR, U4 74HC595D, U5 74HC595D, U6 LTV-847, U7 LTV-847, U8 74HC165, U9 74HC165

Commit message: Add notes to CNC-relays project
Other:
- board text added: "TODO: Cutout for RJ45 is a bit too small TODO: N7803-1PH footprint is wrong Warning: J13 (relay power) is installed backwards"
Changed lines of the file:
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@@
   (gr_line (start 119.38 124.46) (end 120.65 127)
     (stroke (width 0.05) (type default)) (layer "Edge.Cuts"))
+  (gr_text "TODO: Cutout for RJ45 is a bit too small\nTODO: N7803-1PH footprint is wrong\nWarning: J13 (relay power) is installed backwards" (at 76.2 133.35) (layer "Cmts.User")
+    (effects (font (size 1.5 1.5) (thickness 0.3) bold) (justify left bottom))
+  )
   (dimension (type aligned) (layer "Dwgs.User")
     (pts (xy 76.2 39.37) (xy 170.18 39.37))
