File: Stepcraft2-model600/relays/CNC-relays-control-panel/CNC-relays-control-panel.kicad_pcb (KiCad board)
At the start: 2 copper layers, 49.5 x 41.9 mm, 26 parts, among them J1 Conn_01x01, J10 Conn_01x01, J11 Conn_01x01, J2 Conn_01x01, J3 Conn_01x01, J4 Conn_01x01, J5 Conn_01x01, J6 Conn_01x01, J7 Conn_01x01, J8 Conn_01x01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

Commit message: Finish CNC-relays
Other:
- board text added: "TODO ON/OFF are swapped (think about how switches work)"
